File: Kettcar_Control_HW.kicad_sch (KiCad schematic)
At the start: 114 parts, among them J1 Battery 1, J10 WS2812, J11 I²C, J12 Horn, J13 Inputs 2, J14 Outputs 1, J15 Enable Front, J16 Throttle, J17 Brake, J18 Enable Rear, J19 Outputs 2, J2 DC/DC 48V=>24V, J20 UART Front, J21 UART Rear, J3 DC/DC 24V=>5V, J4 Battery 2, J5 Headlights, J6 Battery Out, J7 Battery Out, J8 Indicators, J9 Inputs 1, Q1 AO4407A, Q10 BSS138BKS, Q11 BSS138BKS, Q12 BSS138BKS, Q2 AO4407A, Q3 AO4407A, Q4 AO4407A, Q5 AO4407A, Q6 AO4407A, Q7 MMBT7002K, Q8 IXTP96P085T, Q9 MMBT7002K, U1 NCP114BSN330T1G, U10 CNY17-3, U11 TBD62083A, U12 74HC595, U13 NLAST4599, U14 NLAST4599, U2 TBD62083A, U3 74HC595, U4 Arduino Nano, U5 74HC165, U6 74HC165, U7 TBD62083A, U8 74HC595, U9 CNY17-3

Commit message: Remove "do not populate" status for HW UART components
Parts:
- Q10, R30, R31, R32, R33, U13, U14: now fitted
Changed lines of the file:
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@@
   (title_block
     (title "Kettcar Control")
-    (date "2023-05-23")
+    (date "2023-06-05")
     (rev "1.0")
     (company "xatLabs")
@@
   )
   (symbol (lib_id "custom:Q_DUAL_NMOS_S1G1D2S2G2D1") (at 154.94 256.54 270) (unit 2)
-    (in_bom yes) (on_board yes) (dnp yes) (fields_autoplaced)
+    (in_bom yes) (on_board yes) (dnp no) (fields_autoplaced)
     (property "Reference" "Q10" (at 154.94 264.16 90)
       (effects (font (size 1.27 1.27)))
@@
   )
   (symbol (lib_id "custom:Analog_Switch_SPDT_NLAST4599") (at 99.06 232.41 0) (mirror y) (unit 1)
-    (in_bom yes) (on_board yes) (dnp yes)
+    (in_bom yes) (on_board yes) (dnp no)
     (property "Reference" "U13" (at 99.06 223.52 0)
       (effects (font (size 1.27 1.27)))
@@
       (effects (font (size 1.27 1.27)) hide)
     )
+    (property "Order No." "" (at 99.06 232.41 0)
+      (effects (font (size 1.27 1.27)) hide)
+    )
+    (property "Supplier" "" (at 99.06 232.41 0)
+      (effects (font (size 1.27 1.27)) hide)
+    )
     (pin "1")
     (pin "2")
@@
   )
   (symbol (lib_id "Device:R_Small") (at 162.56 254 0) (mirror y) (unit 1)
-    (in_bom yes) (on_board yes) (dnp yes)
+    (in_bom yes) (on_board yes) (dnp no)
     (property "Reference" "R33" (at 165.1 253.365 0)
       (effects (font (size 1.27 1.27)) (justify right))
@@
       (effects (font (size 1.27 1.27)) hide)
     )
+    (property "Order No." "" (at 162.56 254 0)
+      (effects (font (size 1.27 1.27)) hide)
+    )
+    (property "Supplier" "" (at 162.56 254 0)
+      (effects (font (size 1.27 1.27)) hide)
+    )
     (pin "1")
     (pin "2")
@@
   )
   (symbol (lib_id "custom:Analog_Switch_SPDT_NLAST4599") (at 99.06 250.19 0) (mirror y) (unit 1)
-    (in_bom yes) (on_board yes) (dnp yes)
+    (in_bom yes) (on_board yes) (dnp no)
     (property "Reference" "U14" (at 99.06 241.3 0)
       (effects (font (size 1.27 1.27)))
@@
       (effects (font (size 1.27 1.27)) hide)
     )
+    (property "Order No." "" (at 99.06 250.19 0)
+      (effects (font (size 1.27 1.27)) hide)
+    )
+    (property "Supplier" "" (at 99.06 250.19 0)
+      (effects (font (size 1.27 1.27)) hide)
+    )
     (pin "1")
     (pin "2")
@@
   )
   (symbol (lib_id "Device:R_Small") (at 147.32 254 0) (unit 1)
-    (in_bom yes) (on_board yes) (dnp yes)
+    (in_bom yes) (on_board yes) (dnp no)
     (property "Reference" "R32" (at 144.78 253.365 0)
       (effects (font (size 1.27 1.27)) (justify right))
@@
       (effects (font (size 1.27 1.27)) hide)
     )
+    (property "Order No." "" (at 147.32 254 0)
+      (effects (font (size 1.27 1.27)) hide)
+    )
+    (property "Supplier" "" (at 147.32 254 0)
+      (effects (font (size 1.27 1.27)) hide)
+    )
     (pin "1")
     (pin "2")
@@
   )
   (symbol (lib_id "Device:R_Small") (at 162.56 224.79 0) (mirror y) (unit 1)
-    (in_bom yes) (on_board yes) (dnp yes)
+    (in_bom yes) (on_board yes) (dnp no)
     (property "Reference" "R31" (at 165.1 224.155 0)
       (effects (font (size 1.27 1.27)) (justify right))
@@
       (effects (font (size 1.27 1.27)) hide)
     )
+    (property "Order No." "" (at 162.56 224.79 0)
+      (effects (font (size 1.27 1.27)) hide)
+    )
+    (property "Supplier" "" (at 162.56 224.79 0)
+      (effects (font (size 1.27 1.27)) hide)
+    )
     (pin "1")
     (pin "2")
@@
   )
   (symbol (lib_id "Device:R_Small") (at 147.32 224.79 0) (unit 1)
-    (in_bom yes) (on_board yes) (dnp yes)
+    (in_bom yes) (on_board yes) (dnp no)
     (property "Reference" "R30" (at 144.78 224.155 0)
       (effects (font (size 1.27 1.27)) (justify right))
@@
       (effects (font (size 1.27 1.27)) hide)
     )
+    (property "Order No." "" (at 147.32 224.79 0)
+      (effects (font (size 1.27 1.27)) hide)
+    )
+    (property "Supplier" "" (at 147.32 224.79 0)
+      (effects (font (size 1.27 1.27)) hide)
+    )
     (pin "1")
     (pin "2")
@@
   )
   (symbol (lib_id "custom:Q_DUAL_NMOS_S1G1D2S2G2D1") (at 154.94 227.33 270) (unit 1)
-    (in_bom yes) (on_board yes) (dnp yes) (fields_autoplaced)
+    (in_bom yes) (on_board yes) (dnp no) (fields_autoplaced)
     (property "Reference" "Q10" (at 154.94 234.95 90)
       (effects (font (size 1.27 1.27)))
